File: eagle/littlelights.brd (EAGLE design)
At the start: 21.6 x 10.2 mm, 12 parts, among them U1 Tiny85-20-SMT

Commit message: Added digikey attributes
Parts:
- R1: value 500 -> 470
Changed lines of the file:
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@@
 <?xml version="1.0" encoding="utf-8"?>
 <!DOCTYPE eagle SYSTEM "eagle.dtd">
-<eagle version="7.2.0">
+<eagle version="7.3.0">
 <drawing>
 <settings>
@@
 </autorouter>
 <elements>
-<element name="R1" library="resistor" package="R0603" value="500" x="16.51" y="2.54" rot="R90"/>
+<element name="R1" library="resistor" package="R0603" value="470" x="16.51" y="2.54" rot="R90">
+<attribute name="DIGIKEY" value="MCT0603-470-CFCT-ND" x="16.51" y="2.54" size="1.778" layer="27" rot="R90" display="off"/>
+</element>
 <element name="U1" library="SparkFun-DigitalIC" package="SO08-EIAJ" value="Tiny85-20-SMT" x="10.16" y="3.81" rot="R270">
 <attribute name="PROD_ID" value="IC-09092" x="10.16" y="3.81" size="1.778" layer="27" rot="R270" display="off"/>
+<attribute name="DIGIKEY" value="ATTINY85-20SHRCT-ND" x="10.16" y="3.81" size="1.778" layer="27" rot="R270" display="off"/>
 </element>
 <element name="PRST" library="wirepad" package="SMD1,27-2,54" value="" x="6.35" y="8.89"/>
