File: eagle/4pwm.sch (EAGLE design)
At the start: 17 parts, among them U1 Tiny85-20-SMT

Commit message: Fixed up the labels to match reality
Connections:
- net N$5: now also CH2.P; no longer CH3.P
- net N$6: now also CH3.P; no longer CH2.P
Other:
- moved on the sheet: CH2, CH3
Changed lines of the file:
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@@
 <part name="PPM" library="wirepad" deviceset="SMD2" device=""/>
 <part name="CH1" library="wirepad" deviceset="SMD2" device=""/>
+<part name="CH3" library="wirepad" deviceset="SMD2" device=""/>
 <part name="CH2" library="wirepad" deviceset="SMD2" device=""/>
-<part name="CH3" library="wirepad" deviceset="SMD2" device=""/>
 <part name="CH4" library="wirepad" deviceset="SMD2" device=""/>
 <part name="VCC1" library="wirepad" deviceset="SMD2" device=""/>
@@
 <attribute name="VALUE" x="74.803" y="61.722" size="1.778" layer="96" rot="R180"/>
 </instance>
-<instance part="CH2" gate="1" x="73.66" y="53.34" smashed="yes" rot="R180">
+<instance part="CH3" gate="1" x="73.66" y="53.34" smashed="yes" rot="R180">
 <attribute name="NAME" x="79.883" y="54.0258" size="1.778" layer="95" rot="R180"/>
 <attribute name="VALUE" x="74.803" y="56.642" size="1.778" layer="96" rot="R180"/>
 </instance>
-<instance part="CH3" gate="1" x="73.66" y="55.88" smashed="yes" rot="R180">
+<instance part="CH2" gate="1" x="73.66" y="55.88" smashed="yes" rot="R180">
 <attribute name="NAME" x="79.883" y="56.5658" size="1.778" layer="95" rot="R180"/>
 <attribute name="VALUE" x="74.803" y="59.182" size="1.778" layer="96" rot="R180"/>
@@
 <segment>
 <pinref part="U1" gate="G$1" pin="PB2(SCK/ADC1)"/>
-<pinref part="CH3" gate="1" pin="P"/>
+<pinref part="CH2" gate="1" pin="P"/>
 <wire x1="63.5" y1="55.88" x2="71.12" y2="55.88" width="0.1524" layer="91"/>
 </segment>
@@
 <segment>
 <pinref part="U1" gate="G$1" pin="PB3(ADC3)"/>
-<pinref part="CH2" gate="1" pin="P"/>
+<pinref part="CH3" gate="1" pin="P"/>
 <wire x1="63.5" y1="53.34" x2="71.12" y2="53.34" width="0.1524" layer="91"/>
 </segment>

Commit message: Remove unnecessary reset pullup
Parts:
- removed R1: 10K, SparkFun-Passives:RESISTOR0603-RES
Connections:
- removed net N$1: R1.1, U1.PB5(NRES)
- net VCC: no longer R1.2
Changed lines of the file:
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@@
 <part name="GND3" library="wirepad" deviceset="SMD2" device=""/>
 <part name="GND4" library="wirepad" deviceset="SMD2" device=""/>
-<part name="R1" library="SparkFun-Passives" deviceset="RESISTOR" device="0603-RES" value="10K"/>
 <part name="P+1" library="supply1" deviceset="VCC" device=""/>
 <part name="GND5" library="supply1" deviceset="GND" device=""/>
@@
 <instance part="GND3" gate="1" x="71.12" y="22.86"/>
 <instance part="GND4" gate="1" x="71.12" y="20.32"/>
-<instance part="R1" gate="G$1" x="68.58" y="48.26"/>
 <instance part="P+1" gate="VCC" x="25.4" y="73.66"/>
 <instance part="GND5" gate="1" x="25.4" y="40.64"/>
@@
 <wire x1="35.56" y1="60.96" x2="27.94" y2="60.96" width="0.1524" layer="91"/>
 <pinref part="VCC" gate="1" pin="P"/>
-</segment>
-<segment>
-<pinref part="R1" gate="G$1" pin="2"/>
-<wire x1="73.66" y1="48.26" x2="81.28" y2="48.26" width="0.1524" layer="91"/>
-<label x="81.28" y="48.26" size="1.778" layer="95" rot="R180"/>
 </segment>
 <segment>
@@
 </segment>
 </net>
-<net name="N$1" class="0">
-<segment>
-<pinref part="U1" gate="G$1" pin="PB5(NRES)"/>
-<pinref part="R1" gate="G$1" pin="1"/>
-</segment>
-</net>
